Commit message: started implementing NN Agent

File: link_bot_description/urdf/link_bot.urdf (robot description, URDF)
Before this commit: robot myfirst, 2 links, 1 joints
Links:
- added link head, mass 0.1; collision box size=0.2 0.2 0.2; visual sphere radius=0.1
Joints:
- added joint head_joint: type revolute, parent link_1, child head, origin xyz=1 0 0, axis 0 0 1, limit lower=-2 upper=2 effort=10 velocity=1

Commit message: trying to optimize linear model with TF

File: link_bot_description/urdf/link_bot.urdf (robot description, URDF)
Before this commit: robot myfirst, 3 links, 2 joints
Joints:
- joint head_joint: limit lower=-2 upper=2 effort=10 velocity=1 -> lower=-3 upper=3 effort=10 velocity=1
- joint joint: limit lower=-2 upper=2 effort=10 velocity=1 -> lower=-3 upper=3 effort=10 velocity=1

Commit message: update gazebo sim to generate new data

File: link_bot_description/urdf/link_bot.urdf (robot description, URDF)
Before this commit: robot link_bot, 3 links, 2 joints
Links:
- removed link link_0
- removed link link_1
- added link mid, mass 10; collision box size=0.2 0.2 1; visual cylinder length=1 radius=0.1
- added link tail, mass 10; collision box size=0.2 0.2 1; visual cylinder length=1 radius=0.1
Joints:
- joint head_joint: parent link_1 -> mid
- joint joint: child link_1 -> mid; parent link_0 -> tail
